File: mini-pad-schematic/mini-pad-schematic.kicad_sch (KiCad schematic)
At the start: 14 parts, among them J1 5V_REGULATOR, J2 SPI_OLED, SW1 SW_Push, SW2 SW_Push, SW3 SW_Push, SW4 SW_Push, U1 ATtiny85

Commit message: Added buzzer
Parts:
- added BZ1: Buzzer, symbol Device:Buzzer
- added J3: SPI, symbol Connector_Generic:Conn_02x03_Counter_Clockwise
- renumbered LEFT_POT to LEFT_POT1, RIGHT_POT to RIGHT_POT1
Connections:
- net +5V: now also J3.6 (Pin_6)
- net BUTTONS: now also J3.3 (Pin_3)
- net GND: now also BZ1.2 (+), J3.4 (Pin_4)
- net SCK: now also J3.2 (Pin_2)
- net SDA: now also J3.5 (Pin_5)
- net BUZZER: now reaches U1.6 (PB1)
- net BUZZER: now also BZ1.1 (-), J3.1 (Pin_1)

Commit message: update the pcb design
Parts:
- BZ1: footprint (none) -> Buzzer_Beeper:Buzzer_12x9.5RM7.6
- J1: footprint (none) -> Connector_PinHeader_2.54mm:PinHeader_1x02_P2.54mm_Vertical
- J2: value SPI_OLED -> I2C_OLED; footprint (none) -> Connector_PinSocket_2.54mm:PinSocket_1x04_P2.54mm_Vertical
- J3: footprint (none) -> Connector_PinSocket_2.54mm:PinSocket_2x03_P2.54mm_Vertical
- POT1: renamed from RIGHT_POT1; footprint (none) -> Potentiometer_THT:Potentiometer_Alpha_RD901F-40-00D_Single_Vertical
- POT2: renamed from LEFT_POT1; footprint (none) -> Potentiometer_THT:Potentiometer_Alpha_RD901F-40-00D_Single_Vertical
- R1, R2, R3, R4, R5: footprint (none) -> Resistor_THT:R_Axial_DIN0207_L6.3mm_D2.5mm_P7.62mm_Horizontal
- SW1, SW2, SW3, SW4: footprint (none) -> Button_Switch_THT:SW_PUSH_6mm_H5mm
Connections:
- net +5V: now also J1.2 (Pin_2), J2.2 (Pin_2), J3.3 (Pin_3); no longer J1.1 (Pin_1), J2.3 (Pin_3), J3.6 (Pin_6)
- net BUZZER: now also J3.4 (Pin_4); no longer J3.1 (Pin_1)
- net GND: now also J1.1 (Pin_1), J2.1 (Pin_1), J3.1 (Pin_1); no longer J1.2 (Pin_2), J2.4 (Pin_4), J3.4 (Pin_4)
- net SCK: now also J2.3 (Pin_3), J3.5 (Pin_5); no longer J2.2 (Pin_2), J3.2 (Pin_2)
- net SDA: now also J2.4 (Pin_4), J3.2 (Pin_2); no longer J2.1 (Pin_1), J3.5 (Pin_5)
- net BUTTONS renamed BUTTONS_OUT
- net BUTTONS_OUT: now also J3.6 (Pin_6); no longer J3.3 (Pin_3)
- net LEFT_POT_OUT renamed POT2_OUT
- net RIGHT_POT_OUT renamed POT1_OUT
Other:
- moved on the sheet: J2, J3
